Commit message: update initialization

File: autonomous_exploration_development_environment/vehicle_simulator/urdf/robot.urdf.xacro (robot description, xacro)
@@ -17,10 +17,4 @@
       </geometry>
     </visual>
-    <collision>
-        <geometry>
-          <box size="0.6 0.4 0.3"/>
-        </geometry>
-        <origin xyz="0 0 0" rpy="0 0 0" />
-    </collision>
     <inertial>
       <mass value="1e-5" />
@@ -40,10 +34,4 @@
         <cylinder radius="0.03" length="0.35"/>
       </geometry>
-    <collision>
-        <geometry>
-         <cylinder radius="0.03" length="0.35"/>
-        </geometry>
-        <origin xyz="0 0 0" rpy="0 0 0" />
-    </collision>
     </visual>
     <inertial>
@@ -65,10 +53,4 @@
       </geometry>
     </visual>
-    <collision>
-        <geometry>
-         <cylinder radius="0.15" length="0.1"/>
-        </geometry>
-        <origin xyz="0 0 0" rpy="0 0 0" />
-    </collision>
     <inertial>
       <mass value="1e-5" />
@@ -89,10 +71,4 @@
       </geometry>
     </visual>
-    <collision>
-        <geometry>
-         <cylinder radius="0.15" length="0.1"/>
-        </geometry>
-        <origin xyz="0 0 0" rpy="0 0 0" />
-    </collision>
     <inertial>
       <mass value="1e-5" />
@@ -113,10 +89,4 @@
       </geometry>
     </visual>
-    <collision>
-        <geometry>
-         <cylinder radius="0.15" length="0.1"/>
-        </geometry>
-        <origin xyz="0 0 0" rpy="0 0 0" />
-    </collision>
     <inertial>
       <mass value="1e-5" />
@@ -137,10 +107,4 @@
       </geometry>
     </visual>
-    <collision>
-        <geometry>
-         <cylinder radius="0.15" length="0.1"/>
-        </geometry>
-        <origin xyz="0 0 0" rpy="0 0 0" />
-    </collision>
     <inertial>
       <mass value="1e-5" />
@@ -154,33 +118,4 @@
     <child link="right_rear_wheel"/>
   </joint>
-  <joint name="imu_joint" type="fixed">
-    <origin xyz="0 0 0" rpy="0 0 0" />
-    <parent link="base_origin"/>
-    <child link="imu"/>
-  </joint>
-<link name="imu">
-      <visual>
-          <origin rpy="0 0 0" xyz="0 0 0" />
-          <geometry>
-                  <box size="0.1 0.1 0.1"/>
-          </geometry>
-          <material name= "red" >
-            <color rgba="1.0 0.0 0.0 1.0" />
-          </material>
-      </visual>
-      <collision>
-          <geometry>
-              <box size="0.1 0.1 0.1" />
-          </geometry>
-          <origin xyz="0.0 0.0 0" rpy="0.0 0.0 0.0" />
-      </collision>
-  </link>
-  <xacro:include filename="$(find vehicle_simulator)/urdf/imu.urdf.xacro" />
-  <!--
-  <xacro:include filename="$(find velodyne_description)/urdf/VLP-16.urdf.xacro"/>
-  <xacro:VLP-16 parent="lidar_holder" name="lidar" topic="/velodyne_points" hz="30" samples="1875" gpu="true">
-      <origin xyz="0 0 0.1" rpy="0 0 0" />
-  </xacro:VLP-16>
-  -->
   <xacro:gazebo_material ref="base_link"         color="Red" />
   <xacro:gazebo_material ref="lidar_holder"      color="Black" />
