Commit message: update far_planner

File: sentry_gazebo/urdf/mecanum_base.xacro (robot description, xacro)
@@ -210,7 +210,11 @@
 <!-- modified here -->
   <xacro:include filename="$(find velodyne_description)/urdf/VLP-16.urdf.xacro"/>
-  <xacro:VLP-16 parent="base_link" name="velodyne" topic="/velodyne_points" hz="10" samples="350" min_range="0.5" organize_cloud="true" >
+  <xacro:VLP-16 parent="base_link" name="velodyne" topic="/velodyne_points" hz="5" samples="350" min_range="0.5" organize_cloud="true" >
       <origin xyz="0 0 0.1" rpy="0 0 0" />
   </xacro:VLP-16>
+  <xacro:include filename="$(find sentry_gazebo)/urdf/camera.urdf.xacro"/>
+  <!-- <xacro:camera parent="base_link">
+      <origin xyz="0.1 0 0" rpy="0 0 0" />
+  </xacro:camera>  -->
 <!-- modified here -->
 </robot>
